File: eagle/VCA3+.brd (EAGLE design)
At the start: 100 x 80 mm, 51 parts, among them IC1 TL072P, IC2 TL072P, Q1 2N3906, T2 2N3904, T3 2N3904, T4 2N3904, T5 2N3904, T6 2N3904

Commit message: layout begins
Parts:
- moved R19 129.7 mm to (55.9, 44.5), turned to 90 degrees
- moved OUT 128.2 mm to (66.0, 0.00), turned to 180 degrees
- moved PRESET 123.2 mm to (57.1, 30.5), turned to 90 degrees
- moved OFFSET 121.9 mm to (47.0, 30.5), turned to 270 degrees
- moved R9 119.1 mm to (40.6, 21.6)
- moved GAIN 117.3 mm to (45.7, 3.81)
- moved C13 116.1 mm to (36.8, 30.5), turned to 90 degrees
- moved C4 113.9 mm to (41.9, 55.9), turned to 90 degrees
- moved R13 104.7 mm to (39.4, 30.5), turned to 270 degrees
- moved U$2 103.7 mm to (48.3, 53.3), turned to 180 degrees
- moved R8 99.4 mm to (30.5, 19.1)
- moved R14 99.2 mm to (24.1, 39.4), turned to 180 degrees
- moved C11 99.1 mm to (36.8, 50.8), turned to 90 degrees
- moved R11 98.9 mm to (54.6, 22.9), turned to 180 degrees
- moved U$1 98.0 mm to (48.3, 68.6), turned to 180 degrees
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
Commit message: close to layout
Parts:
- R3: device rcl:0207/10 -> rcl:0207/12
- moved R4 52.1 mm to (43.2, 66.0)
- moved R7 27.2 mm to (29.2, 49.5), turned to 180 degrees
- moved R2 27.1 mm to (41.9, 69.8), turned to 180 degrees
- moved T6 26.9 mm to (39.4, 73.7)
- moved R16 26.2 mm to (26.7, 35.6), turned to 270 degrees
- moved R17 25.1 mm to (21.6, 44.5), turned to 180 degrees
- moved C10 25.0 mm to (45.7, 57.1), turned to 270 degrees
- moved T2 24.3 mm to (33.0, 67.3)
- moved C11 24.1 mm to (44.5, 27.9)
- moved R14 22.9 mm to (47.0, 39.4)
- moved R3 22.5 mm to (52.1, 57.1), turned to 270 degrees
- moved CV-REJ 21.9 mm to (30.5, 44.5), turned to 90 degrees
- moved R12 21.6 mm to (30.5, 57.1), turned to 270 degrees
- moved R18 19.1 mm to (38.1, 44.5), turned to 90 degrees
- moved C4 18.3 mm to (57.1, 66.0), turned to 270 degrees
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Routing:
- net GND: track 0.00 -> 267.9 mm
- net +12V: track 0.00 -> 151.5 mm
- net -12V: track 0.00 -> 137.8 mm
- net N$24: track 0.00 -> 85.0 mm
- net N$8: track 0.00 -> 55.2 mm
- net N$22: track 0.00 -> 47.2 mm
- net N$18: track 0.00 -> 46.1 mm
- net N$11: track 0.00 -> 38.4 mm
- net N$19: track 0.00 -> 23.5 mm
- net N$5: track 0.00 -> 19.8 mm
- net N$25: track 0.00 -> 18.1 mm
- net N$9: track 0.00 -> 17.8 mm
- net N$15: track 0.00 -> 17.6 mm
- net N$17: track 0.00 -> 17.5 mm
- net N$27: track 0.00 -> 11.9 mm
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
Commit message: nearly routed
Parts:
- R3: device rcl:0207/12 -> rcl:0207/10
- moved R15 55.3 mm to (11.4, 49.5)
- moved OFFSET 54.9 mm to (11.4, 71.1)
- moved R19 45.7 mm to (23.5, 57.1)
- moved R11 34.4 mm to (24.1, 27.9), turned to 270 degrees
- moved PRESET 32.0 mm to (27.9, 27.9)
- moved T6 30.0 mm to (15.2, 55.9), turned to 270 degrees
- moved C13 22.9 mm to (35.6, 57.1), turned to 90 degrees
- moved R2 22.2 mm to (47.0, 48.3)
- moved C3 19.4 mm to (26.7, 54.6), turned to 270 degrees
- moved R17 16.5 mm to (38.1, 44.5), turned to 90 degrees
- moved R18 13.0 mm to (25.4, 47.0), turned to 180 degrees
- moved R3 12.8 mm to (50.8, 44.5), turned to 180 degrees
- moved R5 11.7 mm to (11.4, 44.5), turned to 180 degrees
- moved C7 11.5 mm to (8.89, 21.6)
- moved R1 10.2 mm to (10.2, 33.0), turned to 180 degrees
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Routing:
- net +12V: track 151.5 -> 300.5 mm
- net N$24: track 85.0 -> 14.4 mm
- net -12V: track 137.8 -> 67.7 mm
- net N$9: track 17.8 -> 54.1 mm
- net N$8: track 55.2 -> 89.9 mm
- net N$25: track 18.1 -> 49.3 mm
- net N$22: track 47.2 -> 26.3 mm
- net N$21: track 3.81 -> 24.1 mm
- net N$20: track 7.62 -> 20.2 mm
- net N$5: track 19.8 -> 9.42 mm
- net N$11: track 38.4 -> 47.7 mm
- net N$26: track 4.86 -> 12.8 mm
- net GND: track 267.9 -> 261.3 mm
- net N$17: track 17.5 -> 23.8 mm
- net N$27: track 11.9 -> 6.13 mm
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
Commit message: routed
Parts:
- moved C2 25.0 mm to (39.4, 68.6), turned to 90 degrees
- moved PWR1 23.0 mm to (60.3, 44.5)
- moved C5 18.6 mm to (40.0, 63.5), turned to 180 degrees
- moved U$2 18.2 mm to (56.5, 73.7)
- moved C3 15.6 mm to (40.6, 47.6)
- moved OUT 12.7 mm to (66.0, 0.00)
- moved CV 12.1 mm to (36.2, 0.00)
- moved GAIN 11.4 mm to (47.0, 3.81)
- moved R6 10.8 mm to (9.53, 33.7), turned to 270 degrees
- moved AC_IN 8.26 mm to (12.1, 0.00)
- moved DC_IN 8.25 mm to (23.5, 0.00)
- moved R16 7.24 mm to (26.0, 42.5)
- moved R8 6.98 mm to (36.2, 19.1), turned to 180 degrees
- moved R10 6.35 mm to (52.1, 14.0)
- moved R18 4.84 mm to (29.8, 48.9), turned to 90 degrees
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Routing:
- net N$7: track 17.3 -> 88.0 mm
- net GND: track 261.3 -> 319.0 mm
- net -12V: track 67.7 -> 118.3 mm, vias 0 -> 4
- net N$2: track 10.1 -> 46.4 mm
- net N$6: track 5.39 -> 34.3 mm
- net N$14: track 0.00 -> 19.6 mm
- net N$1: track 12.2 -> 30.9 mm
- net N$20: track 20.2 -> 33.9 mm, vias 0 -> 2
- net N$11: track 47.7 -> 34.8 mm
- net N$26: track 12.8 -> 4.02 mm
- net N$4: track 12.0 -> 3.81 mm
- net N$3: track 0.00 -> 6.62 mm
- net N$9: track 54.1 -> 49.5 mm
- net N$18: track 46.6 -> 41.9 mm
- net N$22: track 26.3 -> 30.8 mm
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
Commit message: cutout
Parts:
- moved C10 4.26 mm to (48.3, 59.1)
- moved R8 3.81 mm to (32.4, 19.1)
- moved OUT 2.54 mm to (63.5, 0.00)
- moved PWR1 2.54 mm to (57.8, 44.5)
- moved U$1 2.54 mm to (57.8, 71.1)
- moved DC_IN 2.54 mm to (21.0, 0.00)
- moved PRESET 2.54 mm to (25.4, 29.2)
- moved Q1 2.54 mm to (24.1, 66.0)
- moved R17 2.54 mm to (31.1, 43.2)
- moved T3 2.54 mm to (14.0, 71.1)
- moved T6 2.54 mm to (12.7, 55.9)
- moved C7 2.54 mm to (4.45, 22.2)
- moved R1 2.54 mm to (4.45, 33.7)
- moved R6 2.54 mm to (6.99, 33.7)
- moved AC_IN 2.54 mm to (9.53, 0.00)
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Routing:
- net +12V: track 298.6 -> 296.9 mm
- net N$18: track 41.9 -> 42.9 mm
- net N$22: track 30.8 -> 31.5 mm
- net N$2: track 46.4 -> 45.8 mm
- net N$24: track 14.7 -> 14.1 mm
- net -12V: track 118.3 -> 118.8 mm
- net N$14: track 19.6 -> 19.1 mm
Other:
- board size 100 x 80 mm -> 100.9 x 80.9 mm
